File: circuitry/PCB/PCB.kicad_sch (KiCad schematic)
At the start: 77 parts, among them J1 K-LC5, J2 ADS1115, J3 I/Q-amp, J4 Raspberry_Pi_2_3, SW1 SW_SPDT, U1 MCP6022, U2 AP2139AK-3.3TRG1, U3 MCP6022, U4 MCP6022, U5 MCP6022

Commit message: just pushing final board design for future reference
Parts:
- removed C16, C27: 4.7u, Capacitor_SMD:C_1206_3216Metric_Pad1.33x1.80mm_HandSolder, symbol Device:C_Small
- C10, C11, C17, C18, C24, C25, C4, C5: footprint Capacitor_THT:CP_Radial_D8.0mm_P2.50mm -> Capacitor_Tantalum_SMD:CP_EIA-3528-12_Kemet-T_Pad1.50x2.35mm_HandSolder
- C3: value 4.7u -> 1u
- I1: renamed from TP1; footprint TestPoint:TestPoint_Pad_D3.0mm -> TestPoint:TestPoint_Pad_D2.5mm
- I2: renamed from TP5; footprint TestPoint:TestPoint_Pad_D3.0mm -> TestPoint:TestPoint_Pad_D2.5mm
- Q1: renamed from TP2; footprint TestPoint:TestPoint_Pad_D3.0mm -> TestPoint:TestPoint_Pad_D2.5mm
- Q2: renamed from TP6; footprint TestPoint:TestPoint_Pad_D3.0mm -> TestPoint:TestPoint_Pad_D2.5mm
- SW1: footprint (none) -> Proj_Lib:PCM12SMTR
- TP3, TP4, TP7, TP8: footprint TestPoint:TestPoint_Pad_D3.0mm -> TestPoint:TestPoint_Pad_D2.5mm
Connections:
- net 5V: now also J4.4 (5V)
- net GND: now also J3.3 (GND), J3.4 (GND), J4.14 (GND), J4.20 (GND), J4.25 (GND), J4.30 (GND), J4.34 (GND), J4.39 (GND), J4.6 (GND)
- net I: now also C4.2; no longer C5.2
- net I_amp: now also C30.1, J2.7 (A0), J3.1 (I_amp), U5.1, U5.2 (-); no longer C31.1, J2.8 (A1), J3.2 (I_amp), U5.6 (-), U5.7
- net Q: now also C5.2; no longer C4.2
- net Q_amp: now also C31.1, J2.8 (A1), J3.2 (Q_amp), U5.6 (-), U5.7; no longer C30.1, J2.7 (A0), J3.1 (Q_amp), U5.1, U5.2 (-)
- no-connect marks 44 -> 36
Other:
- moved on the sheet: C20
